File: hardware/Multipro-txV2-NRF24.sch (KiCad schematic (older format))
At the start: 30 parts, among them J1 AVR-ISP-6, J2 Conn_01x05, SW1 SW_Coded_SH-7050, SW2 SW_Push, SW3 SW_Push, U1 LM317_3PinPackage, U2 ATmega328-AU, U3 NRF24L01 G-24 Breakout, Y1 16MHz

Commit message: values update
Parts:
- D1: value LED -> LED GREEN
- R3: value 1k -> 1k5
- R6: value 10k -> 2k2
Changed lines of the file:
@@
 EESchema Schematic File Version 4
+LIBS:Multipro-txV2-NRF24-cache
 EELAYER 30 0
 EELAYER END
@@
 P 3500 3300
 F 0 "R3" H 3570 3346 50  0000 L CNN
-F 1 "1k" H 3570 3255 50  0000 L CNN
+F 1 "1k5" H 3570 3255 50  0000 L CNN
 F 2 "obbo_footprints:R_0805K" V 3430 3300 50  0001 C CNN
 F 3 "~" H 3500 3300 50  0001 C CNN
@@
 P 7200 4750
 F 0 "R6" H 7270 4796 50  0000 L CNN
-F 1 "10k" H 7270 4705 50  0000 L CNN
+F 1 "2k2" H 7270 4705 50  0000 L CNN
 F 2 "obbo_footprints:R_0805K" V 7130 4750 50  0001 C CNN
 F 3 "~" H 7200 4750 50  0001 C CNN
@@
 P 3900 3600
 F 0 "D1" H 3893 3345 50  0000 C CNN
-F 1 "LED" H 3893 3436 50  0000 C CNN
+F 1 "LED GREEN" H 3893 3436 50  0000 C CNN
 F 2 "LED_SMD:LED_0805_2012Metric_Pad1.15x1.40mm_HandSolder" H 3900 3600 50  0001 C CNN
 F 3 "~" H 3900 3600 50  0001 C CNN
